Commit message: modified path to meshes

File: models/iCubGazeboV2_5/model.urdf (robot description, URDF)
Before this commit: robot iCub, 189 links, 188 joints
Links:
- link chest: geometry collision mesh filename=ABSOLUTE_PATH_TO_MESHES/simmechanics/sim_sea_2-5_chest_bb_p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 scale=0.001 0.001 0.001; visual mesh filename=ABSOLUTE_PATH_TO_MESHES/simmechanics/sim_sea_2-5_chest_bb_p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 scale=0.001 0.001 0.001
- link head: geometry collision mesh filename=ABSOLUTE_PATH_TO_MESHES/simmechanics/sim_sea_2-5_head_prt-b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 scale=0.001 0.001 0.001; visual mesh filename=ABSOLUTE_PATH_TO_MESHES/simmechanics/sim_sea_2-5_head_prt-b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 scale=0.001 0.001 0.001
- link l_ankle_1: geometry collision mesh filename=ABSOLUTE_PATH_TO_MESHES/simmechanics/sim_sea_2-5_l_ankle_pr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 scale=0.001 0.001 0.001; visual mesh filename=ABSOLUTE_PATH_TO_MESHES/simmechanics/sim_sea_2-5_l_ankle_pr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 scale=0.001 0.001 0.001
- link l_ankle_2: geometry collision mesh filename=ABSOLUTE_PATH_TO_MESHES/simmechanics/sim_sea_2-5_l_foot_prt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 scale=0.001 0.001 0.001; visual mesh filename=ABSOLUTE_PATH_TO_MESHES/simmechanics/sim_sea_2-5_l_foot_prt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 scale=0.001 0.001 0.001
- link l_elbow_1: geometry collision mesh filename=ABSOLUTE_PATH_TO_MESHES/simmechanics/sim_sea_2-5_l_elbow_pr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 scale=0.001 0.001 0.001; visual mesh filename=ABSOLUTE_PATH_TO_MESHES/simmechanics/sim_sea_2-5_l_elbow_pr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 scale=0.001 0.001 0.001
- link l_foot: geometry collision box size=0.16 0.072 0.001; visual mesh filename=ABSOLUTE_PATH_TO_MESHES/simmechanics/sim_sea_2-5_l_sole_prt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 scale=0.001 0.001 0.001
- link l_forearm: geometry collision mesh filename=ABSOLUTE_PATH_TO_MESHES/simmechanics/sim_sea_2-5_l_forearm_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 scale=0.001 0.001 0.001; visual mesh filename=ABSOLUTE_PATH_TO_MESHES/simmechanics/sim_sea_2-5_l_forearm_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 scale=0.001 0.001 0.001
- link l_hand: geometry collision mesh filename=ABSOLUTE_PATH_TO_MESHES/simmechanics/sim_sea_2-5_l_hand_prt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 scale=0.001 0.001 0.001; visual mesh filename=ABSOLUTE_PATH_TO_MESHES/simmechanics/sim_sea_2-5_l_hand_prt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 scale=0.001 0.001 0.001
- link l_hip_1: geometry collision mesh filename=ABSOLUTE_PATH_TO_MESHES/simmechanics/sim_sea_2-5_l_hip_1_pr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 scale=0.001 0.001 0.001; visual mesh filename=ABSOLUTE_PATH_TO_MESHES/simmechanics/sim_sea_2-5_l_hip_1_pr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 scale=0.001 0.001 0.001
- link l_hip_2: geometry collision mesh filename=ABSOLUTE_PATH_TO_MESHES/simmechanics/sim_sea_2-5_l_hip_2_pr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 scale=0.001 0.001 0.001; visual mesh filename=ABSOLUTE_PATH_TO_MESHES/simmechanics/sim_sea_2-5_l_hip_2_pr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 scale=0.001 0.001 0.001
- link l_hip_3: geometry collision mesh filename=ABSOLUTE_PATH_TO_MESHES/simmechanics/sim_sea_2-5_l_upper_th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 scale=0.001 0.001 0.001; visual mesh filename=ABSOLUTE_PATH_TO_MESHES/simmechanics/sim_sea_2-5_l_upper_th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 scale=0.001 0.001 0.001
- link l_lower_leg: geometry collision mesh filename=ABSOLUTE_PATH_TO_MESHES/simmechanics/sim_sea_2-5_l_shank_pr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 scale=0.001 0.001 0.001; visual mesh filename=ABSOLUTE_PATH_TO_MESHES/simmechanics/sim_sea_2-5_l_shank_pr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 scale=0.001 0.001 0.001
- link l_shoulder_1: geometry collision mesh filename=ABSOLUTE_PATH_TO_MESHES/simmechanics/sim_sea_2-5_l_shoulder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 scale=0.001 0.001 0.001; visual mesh filename=ABSOLUTE_PATH_TO_MESHES/simmechanics/sim_sea_2-5_l_shoulder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 scale=0.001 0.001 0.001
- link l_shoulder_2: geometry collision mesh filename=ABSOLUTE_PATH_TO_MESHES/simmechanics/sim_sea_2-5_l_shoulder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 scale=0.001 0.001 0.001; visual mesh filename=ABSOLUTE_PATH_TO_MESHES/simmechanics/sim_sea_2-5_l_shoulder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 scale=0.001 0.001 0.001
- link l_shoulder_3: geometry collision mesh filename=ABSOLUTE_PATH_TO_MESHES/simmechanics/sim_sea_2-5_l_upper_ar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 scale=0.001 0.001 0.001; visual mesh filename=ABSOLUTE_PATH_TO_MESHES/simmechanics/sim_sea_2-5_l_upper_ar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 scale=0.001 0.001 0.001
- link l_upper_arm: geometry collision mesh filename=ABSOLUTE_PATH_TO_MESHES/simmechanics/sim_sea_2-5_l_elbow_pr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 scale=0.001 0.001 0.001; visual mesh filename=ABSOLUTE_PATH_TO_MESHES/simmechanics/sim_sea_2-5_l_elbow_pr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 scale=0.001 0.001 0.001
- link l_upper_leg: geometry collision mesh filename=ABSOLUTE_PATH_TO_MESHES/simmechanics/sim_sea_2-5_l_thigh_pr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 scale=0.001 0.001 0.001; visual mesh filename=ABSOLUTE_PATH_TO_MESHES/simmechanics/sim_sea_2-5_l_thigh_pr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 scale=0.001 0.001 0.001
- link l_wrist_1: geometry collision mesh filename=ABSOLUTE_PATH_TO_MESHES/simmechanics/sim_sea_2-5_l_wrist_pi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 scale=0.001 0.001 0.001; visual mesh filename=ABSOLUTE_PATH_TO_MESHES/simmechanics/sim_sea_2-5_l_wrist_pi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 scale=0.001 0.001 0.001
- link neck_1: geometry collision mesh filename=ABSOLUTE_PATH_TO_MESHES/simmechanics/sim_sea_2-5_neck_1_prt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 scale=0.001 0.001 0.001; visual mesh filename=ABSOLUTE_PATH_TO_MESHES/simmechanics/sim_sea_2-5_neck_1_prt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 scale=0.001 0.001 0.001
- link neck_2: geometry collision mesh filename=ABSOLUTE_PATH_TO_MESHES/simmechanics/sim_sea_2-5_neck_2_prt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 scale=0.001 0.001 0.001; visual mesh filename=ABSOLUTE_PATH_TO_MESHES/simmechanics/sim_sea_2-5_neck_2_prt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 scale=0.001 0.001 0.001
- link r_ankle_1: geometry collision mesh filename=ABSOLUTE_PATH_TO_MESHES/simmechanics/sim_sea_2-5_r_ankle_pr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 scale=0.001 0.001 0.001; visual mesh filename=ABSOLUTE_PATH_TO_MESHES/simmechanics/sim_sea_2-5_r_ankle_pr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 scale=0.001 0.001 0.001
- link r_ankle_2: geometry collision mesh filename=ABSOLUTE_PATH_TO_MESHES/simmechanics/sim_sea_2-5_r_foot_prt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 scale=0.001 0.001 0.001; visual mesh filename=ABSOLUTE_PATH_TO_MESHES/simmechanics/sim_sea_2-5_r_foot_prt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 scale=0.001 0.001 0.001
- link r_elbow_1: geometry collision mesh filename=ABSOLUTE_PATH_TO_MESHES/simmechanics/sim_sea_2-5_r_elbow_pr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 scale=0.001 0.001 0.001; visual mesh filename=ABSOLUTE_PATH_TO_MESHES/simmechanics/sim_sea_2-5_r_elbow_pr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 scale=0.001 0.001 0.001
- link r_foot: geometry collision box size=0.16 0.072 0.001; visual mesh filename=ABSOLUTE_PATH_TO_MESHES/simmechanics/sim_sea_2-5_r_sole_prt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 scale=0.001 0.001 0.001
- link r_forearm: geometry collision mesh filename=ABSOLUTE_PATH_TO_MESHES/simmechanics/sim_sea_2-5_r_forearm_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 scale=0.001 0.001 0.001; visual mesh filename=ABSOLUTE_PATH_TO_MESHES/simmechanics/sim_sea_2-5_r_forearm_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 scale=0.001 0.001 0.001
- link r_hand: geometry collision mesh filename=ABSOLUTE_PATH_TO_MESHES/simmechanics/sim_sea_2-5_r_hand_prt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 scale=0.001 0.001 0.001; visual mesh filename=ABSOLUTE_PATH_TO_MESHES/simmechanics/sim_sea_2-5_r_hand_prt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 scale=0.001 0.001 0.001
- link r_hip_1: geometry collision mesh filename=ABSOLUTE_PATH_TO_MESHES/simmechanics/sim_sea_2-5_r_hip_1_pr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 scale=0.001 0.001 0.001; visual mesh filename=ABSOLUTE_PATH_TO_MESHES/simmechanics/sim_sea_2-5_r_hip_1_pr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 scale=0.001 0.001 0.001
- link r_hip_2: geometry collision mesh filename=ABSOLUTE_PATH_TO_MESHES/simmechanics/sim_sea_2-5_r_hip_2_pr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 scale=0.001 0.001 0.001; visual mesh filename=ABSOLUTE_PATH_TO_MESHES/simmechanics/sim_sea_2-5_r_hip_2_pr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 scale=0.001 0.001 0.001
- link r_hip_3: geometry collision mesh filename=ABSOLUTE_PATH_TO_MESHES/simmechanics/sim_sea_2-5_r_upper_th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 scale=0.001 0.001 0.001; visual mesh filename=ABSOLUTE_PATH_TO_MESHES/simmechanics/sim_sea_2-5_r_upper_th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 scale=0.001 0.001 0.001
- link r_lower_leg: geometry collision mesh filename=ABSOLUTE_PATH_TO_MESHES/simmechanics/sim_sea_2-5_r_shank_pr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 scale=0.001 0.001 0.001; visual mesh filename=ABSOLUTE_PATH_TO_MESHES/simmechanics/sim_sea_2-5_r_shank_pr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 scale=0.001 0.001 0.001
- link r_shoulder_1: geometry collision mesh filename=ABSOLUTE_PATH_TO_MESHES/simmechanics/sim_sea_2-5_r_shoulder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 scale=0.001 0.001 0.001; visual mesh filename=ABSOLUTE_PATH_TO_MESHES/simmechanics/sim_sea_2-5_r_shoulder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 scale=0.001 0.001 0.001
- link r_shoulder_2: geometry collision mesh filename=ABSOLUTE_PATH_TO_MESHES/simmechanics/sim_sea_2-5_r_shoulder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 scale=0.001 0.001 0.001; visual mesh filename=ABSOLUTE_PATH_TO_MESHES/simmechanics/sim_sea_2-5_r_shoulder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 scale=0.001 0.001 0.001
- link r_shoulder_3: geometry collision mesh filename=ABSOLUTE_PATH_TO_MESHES/simmechanics/sim_sea_2-5_r_upper_ar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 scale=0.001 0.001 0.001; visual mesh filename=ABSOLUTE_PATH_TO_MESHES/simmechanics/sim_sea_2-5_r_upper_ar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 scale=0.001 0.001 0.001
- link r_upper_arm: geometry collision mesh filename=ABSOLUTE_PATH_TO_MESHES/simmechanics/sim_sea_2-5_r_elbow_pr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 scale=0.001 0.001 0.001; visual mesh filename=ABSOLUTE_PATH_TO_MESHES/simmechanics/sim_sea_2-5_r_elbow_pr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 scale=0.001 0.001 0.001
- link r_upper_leg: geometry collision mesh filename=ABSOLUTE_PATH_TO_MESHES/simmechanics/sim_sea_2-5_r_thigh_pr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 scale=0.001 0.001 0.001; visual mesh filename=ABSOLUTE_PATH_TO_MESHES/simmechanics/sim_sea_2-5_r_thigh_pr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 scale=0.001 0.001 0.001
- link r_wrist_1: geometry collision mesh filename=ABSOLUTE_PATH_TO_MESHES/simmechanics/sim_sea_2-5_r_wrist_pi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 scale=0.001 0.001 0.001; visual mesh filename=ABSOLUTE_PATH_TO_MESHES/simmechanics/sim_sea_2-5_r_wrist_pi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 scale=0.001 0.001 0.001
- link root_link: geometry collision mesh filename=ABSOLUTE_PATH_TO_MESHES/simmechanics/sim_sea_2-5_root_link_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 scale=0.001 0.001 0.001; visual mesh filename=ABSOLUTE_PATH_TO_MESHES/simmechanics/sim_sea_2-5_root_link_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 scale=0.001 0.001 0.001
- link torso_1: geometry collision mesh filename=ABSOLUTE_PATH_TO_MESHES/simmechanics/sim_sea_2-5_lap_belt_1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 scale=0.001 0.001 0.001; visual mesh filename=ABSOLUTE_PATH_TO_MESHES/simmechanics/sim_sea_2-5_lap_belt_1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 scale=0.001 0.001 0.001
- link torso_2: geometry collision mesh filename=ABSOLUTE_PATH_TO_MESHES/simmechanics/sim_sea_2-5_lap_belt_2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 scale=0.001 0.001 0.001; visual mesh filename=ABSOLUTE_PATH_TO_MESHES/simmechanics/sim_sea_2-5_lap_belt_2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 scale=0.001 0.001 0.001

File: models/icubGazeboSim/model.urdf (robot description, URDF)
Before this commit: robot iCub, 56 links, 55 joints
Links:
- link chest: geometry collision mesh filename=ABSOLUTE_PATH_TO_MESHES/icub_simple_collision_chest.dae scale=1 1 1; visual mesh filename=ABSOLUTE_PATH_TO_MESHES/icub_simple_collision_chest.dae scale=1 1 1
- link head: geometry collision mesh filename=ABSOLUTE_PATH_TO_MESHES/icub_simple_collision_head.dae scale=1 1 1; visual mesh filename=ABSOLUTE_PATH_TO_MESHES/icub_simple_collision_head.dae scale=1 1 1
- link l_ankle_1: geometry collision mesh filename=ABSOLUTE_PATH_TO_MESHES/icub_simple_collision_l_ankle_1.dae scale=1 1 1; visual mesh filename=ABSOLUTE_PATH_TO_MESHES/icub_simple_collision_l_ankle_1.dae scale=1 1 1
- link l_foot: geometry collision mesh filename=ABSOLUTE_PATH_TO_MESHES/icub_simple_collision_l_foot.dae scale=1 1 1; visual mesh filename=ABSOLUTE_PATH_TO_MESHES/icub_simple_collision_l_foot.dae scale=1 1 1
- link l_forearm: geometry collision mesh filename=ABSOLUTE_PATH_TO_MESHES/icub_simple_collision_l_forearm.dae scale=1 1 1; visual mesh filename=ABSOLUTE_PATH_TO_MESHES/icub_simple_collision_l_forearm.dae scale=1 1 1
- link l_hand: geometry collision mesh filename=ABSOLUTE_PATH_TO_MESHES/icub_simple_collision_l_hand.dae scale=1 1 1; visual mesh filename=ABSOLUTE_PATH_TO_MESHES/icub_simple_collision_l_hand.dae scale=1 1 1
- link l_hip_1: geometry collision mesh filename=ABSOLUTE_PATH_TO_MESHES/icub_simple_collision_l_hip_1.dae scale=1 1 1; visual mesh filename=ABSOLUTE_PATH_TO_MESHES/icub_simple_collision_l_hip_1.dae scale=1 1 1
- link l_hip_2: geometry collision mesh filename=ABSOLUTE_PATH_TO_MESHES/icub_simple_collision_l_hip_2.dae scale=1 1 1; visual mesh filename=ABSOLUTE_PATH_TO_MESHES/icub_simple_collision_l_hip_2.dae scale=1 1 1
- link l_lower_leg: geometry collision mesh filename=ABSOLUTE_PATH_TO_MESHES/icub_simple_collision_l_shank.dae scale=1 1 1; visual mesh filename=ABSOLUTE_PATH_TO_MESHES/icub_simple_collision_l_shank.dae scale=1 1 1
- link l_shoulder_1: geometry collision mesh filename=ABSOLUTE_PATH_TO_MESHES/icub_simple_collision_l_shoulder_1.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 scale=1 1 1; visual mesh filename=ABSOLUTE_PATH_TO_MESHES/icub_simple_collision_l_shoulder_1.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 scale=1 1 1
- link l_shoulder_2: geometry collision mesh filename=ABSOLUTE_PATH_TO_MESHES/icub_simple_collision_l_shoulder_2.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 scale=1 1 1; visual mesh filename=ABSOLUTE_PATH_TO_MESHES/icub_simple_collision_l_shoulder_2.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 scale=1 1 1
- link l_upper_arm: geometry collision mesh filename=ABSOLUTE_PATH_TO_MESHES/icub_simple_collision_l_arm.dae scale=1 1 1; visual mesh filename=ABSOLUTE_PATH_TO_MESHES/icub_simple_collision_l_arm.dae scale=1 1 1
- link l_upper_leg: geometry collision mesh filename=ABSOLUTE_PATH_TO_MESHES/icub_simple_collision_l_thigh.dae scale=1 1 1; visual mesh filename=ABSOLUTE_PATH_TO_MESHES/icub_simple_collision_l_thigh.dae scale=1 1 1
- link neck_1: geometry collision mesh filename=ABSOLUTE_PATH_TO_MESHES/icub_simple_collision_neck_1.dae scale=1 1 1; visual mesh filename=ABSOLUTE_PATH_TO_MESHES/icub_simple_collision_neck_1.dae scale=1 1 1
- link neck_2: geometry collision mesh filename=ABSOLUTE_PATH_TO_MESHES/icub_simple_collision_neck_2.dae scale=1 1 1; visual mesh filename=ABSOLUTE_PATH_TO_MESHES/icub_simple_collision_neck_2.dae scale=1 1 1
- link r_ankle_1: geometry collision mesh filename=ABSOLUTE_PATH_TO_MESHES/icub_simple_collision_r_ankle_1.dae scale=1 1 1; visual mesh filename=ABSOLUTE_PATH_TO_MESHES/icub_simple_collision_r_ankle_1.dae scale=1 1 1
- link r_foot: geometry collision mesh filename=ABSOLUTE_PATH_TO_MESHES/icub_simple_collision_r_foot.dae scale=1 1 1; visual mesh filename=ABSOLUTE_PATH_TO_MESHES/icub_simple_collision_r_foot.dae scale=1 1 1
- link r_forearm: geometry collision mesh filename=ABSOLUTE_PATH_TO_MESHES/icub_simple_collision_r_forearm.dae scale=1 1 1; visual mesh filename=ABSOLUTE_PATH_TO_MESHES/icub_simple_collision_r_forearm.dae scale=1 1 1
- link r_hand: geometry collision mesh filename=ABSOLUTE_PATH_TO_MESHES/icub_simple_collision_r_hand.dae scale=1 1 1; visual mesh filename=ABSOLUTE_PATH_TO_MESHES/icub_simple_collision_r_hand.dae scale=1 1 1
- link r_hip_1: geometry collision mesh filename=ABSOLUTE_PATH_TO_MESHES/icub_simple_collision_r_hip_1.dae scale=1 1 1; visual mesh filename=ABSOLUTE_PATH_TO_MESHES/icub_simple_collision_r_hip_1.dae scale=1 1 1
- link r_hip_2: geometry collision mesh filename=ABSOLUTE_PATH_TO_MESHES/icub_simple_collision_r_hip_2.dae scale=1 1 1; visual mesh filename=ABSOLUTE_PATH_TO_MESHES/icub_simple_collision_r_hip_2.dae scale=1 1 1
- link r_lower_leg: geometry collision mesh filename=ABSOLUTE_PATH_TO_MESHES/icub_simple_collision_r_shank.dae scale=1 1 1; visual mesh filename=ABSOLUTE_PATH_TO_MESHES/icub_simple_collision_r_shank.dae scale=1 1 1
- link r_shoulder_1: geometry collision mesh filename=ABSOLUTE_PATH_TO_MESHES/icub_simple_collision_r_shoulder_1.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 scale=1 1 1; visual mesh filename=ABSOLUTE_PATH_TO_MESHES/icub_simple_collision_r_shoulder_1.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 scale=1 1 1
- link r_shoulder_2: geometry collision mesh filename=ABSOLUTE_PATH_TO_MESHES/icub_simple_collision_r_shoulder_2.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 scale=1 1 1; visual mesh filename=ABSOLUTE_PATH_TO_MESHES/icub_simple_collision_r_shoulder_2.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 scale=1 1 1
- link r_upper_arm: geometry collision mesh filename=ABSOLUTE_PATH_TO_MESHES/icub_simple_collision_r_arm.dae scale=1 1 1; visual mesh filename=ABSOLUTE_PATH_TO_MESHES/icub_simple_collision_r_arm.dae scale=1 1 1
- link r_upper_leg: geometry collision mesh filename=ABSOLUTE_PATH_TO_MESHES/icub_simple_collision_r_thigh.dae scale=1 1 1; visual mesh filename=ABSOLUTE_PATH_TO_MESHES/icub_simple_collision_r_thigh.dae scale=1 1 1
- link root_link: geometry collision mesh filename=ABSOLUTE_PATH_TO_MESHES/icub_simple_collision_root_link.dae scale=1 1 1; visual mesh filename=ABSOLUTE_PATH_TO_MESHES/icub_simple_collision_root_link.dae scale=1 1 1
- link torso_1: geometry collision mesh filename=ABSOLUTE_PATH_TO_MESHES/icub_simple_collision_lap_belt_1.dae scale=1 1 1; visual mesh filename=ABSOLUTE_PATH_TO_MESHES/icub_simple_collision_lap_belt_1.dae scale=1 1 1
