Commit message: modified path to meshes

File: models/ironBot/model.urdf (robot description, URDF)
Before this commit: robot iCub, 151 links, 150 joints
Links:
- link chest: geometry collision mesh filename=ABSOLUTE_PATH_TO_MESHES/sim_sea_2-5_chest_bb_prt-binary.dae scale=0.001 0.001 0.001; visual mesh filename=ABSOLUTE_PATH_TO_MESHES/sim_sea_2-5_chest_bb_prt-binary.dae scale=0.001 0.001 0.001
- link chest_l_jet_turbine: geometry collision mesh filename=ABSOLUTE_PATH_TO_TURBINES_MESHES/chest_l_jet_turbine.dae scale=0.001 0.001 0.001; visual mesh filename=ABSOLUTE_PATH_TO_TURBINES_MESHES/chest_l_jet_turbine.dae scale=0.001 0.001 0.001
- link chest_l_jet_turbine_prime: geometry collision mesh filename=ABSOLUTE_PATH_TO_TURBINES_MESHES/chest_l_jet_turbine.dae scale=0.001 0.001 0.001; visual mesh filename=ABSOLUTE_PATH_TO_TURBINES_MESHES/chest_l_jet_turbine.dae scale=0.001 0.001 0.001
- link chest_r_jet_turbine: geometry collision mesh filename=ABSOLUTE_PATH_TO_TURBINES_MESHES/chest_r_jet_turbine.dae scale=0.001 0.001 0.001; visual mesh filename=ABSOLUTE_PATH_TO_TURBINES_MESHES/chest_r_jet_turbine.dae scale=0.001 0.001 0.001
- link chest_r_jet_turbine_prime: geometry collision mesh filename=ABSOLUTE_PATH_TO_TURBINES_MESHES/chest_r_jet_turbine.dae scale=0.001 0.001 0.001; visual mesh filename=ABSOLUTE_PATH_TO_TURBINES_MESHES/chest_r_jet_turbine.dae scale=0.001 0.001 0.001
- link head: geometry collision mesh filename=ABSOLUTE_PATH_TO_MESHES/sim_sea_2-5_head_prt-binary.dae scale=0.001 0.001 0.001; visual mesh filename=ABSOLUTE_PATH_TO_MESHES/sim_sea_2-5_head_prt-binary.dae scale=0.001 0.001 0.001
- link l_ankle_1: geometry collision mesh filename=ABSOLUTE_PATH_TO_MESHES/sim_sea_2-5_l_ankle_prt-binary.dae scale=0.001 0.001 0.001; visual mesh filename=ABSOLUTE_PATH_TO_MESHES/sim_sea_2-5_l_ankle_prt-binary.dae scale=0.001 0.001 0.001
- link l_ankle_2: geometry collision mesh filename=ABSOLUTE_PATH_TO_MESHES/sim_sea_2-5_l_foot_prt-binary.dae scale=0.001 0.001 0.001; visual mesh filename=ABSOLUTE_PATH_TO_MESHES/sim_sea_2-5_l_foot_prt-binary.dae scale=0.001 0.001 0.001
- link l_arm_jet_turbine: geometry collision mesh filename=ABSOLUTE_PATH_TO_TURBINES_MESHES/l_arm_jet_turbine.dae scale=0.001 0.001 0.001; visual mesh filename=ABSOLUTE_PATH_TO_TURBINES_MESHES/l_arm_jet_turbine.dae scale=0.001 0.001 0.001
- link l_arm_jet_turbine_prime: geometry collision mesh filename=ABSOLUTE_PATH_TO_TURBINES_MESHES/l_arm_jet_turbine.dae scale=0.001 0.001 0.001; visual mesh filename=ABSOLUTE_PATH_TO_TURBINES_MESHES/l_arm_jet_turbine.dae scale=0.001 0.001 0.001
- link l_elbow_1: geometry collision mesh filename=ABSOLUTE_PATH_TO_MESHES/sim_sea_2-5_l_elbow_prosup_prt-bina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 scale=0.001 0.001 0.001; visual mesh filename=ABSOLUTE_PATH_TO_MESHES/sim_sea_2-5_l_elbow_prosup_prt-bina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 scale=0.001 0.001 0.001
- link l_foot: geometry collision box size=0.16 0.072 0.001; visual mesh filename=ABSOLUTE_PATH_TO_MESHES/sim_sea_2-5_l_sole_prt-binary.dae scale=0.001 0.001 0.001
- link l_forearm: geometry collision mesh filename=ABSOLUTE_PATH_TO_MESHES/sim_sea_2-5_l_forearm_prt-binary.dae scale=0.001 0.001 0.001; visual mesh filename=ABSOLUTE_PATH_TO_MESHES/sim_sea_2-5_l_forearm_prt-binary.dae scale=0.001 0.001 0.001
- link l_hand: geometry collision mesh filename=ABSOLUTE_PATH_TO_MESHES/sim_sea_2-5_l_hand_prt-binary.dae scale=0.001 0.001 0.001; visual mesh filename=ABSOLUTE_PATH_TO_MESHES/sim_sea_2-5_l_hand_prt-binary.dae scale=0.001 0.001 0.001
- link l_hip_1: geometry collision mesh filename=ABSOLUTE_PATH_TO_MESHES/sim_sea_2-5_l_hip_1_prt-binary.dae scale=0.001 0.001 0.001; visual mesh filename=ABSOLUTE_PATH_TO_MESHES/sim_sea_2-5_l_hip_1_prt-binary.dae scale=0.001 0.001 0.001
- link l_hip_2: geometry collision mesh filename=ABSOLUTE_PATH_TO_MESHES/sim_sea_2-5_l_hip_2_prt-binary.dae scale=0.001 0.001 0.001; visual mesh filename=ABSOLUTE_PATH_TO_MESHES/sim_sea_2-5_l_hip_2_prt-binary.dae scale=0.001 0.001 0.001
- link l_hip_3: geometry collision mesh filename=ABSOLUTE_PATH_TO_MESHES/sim_sea_2-5_l_upper_thigh_prt-binar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 scale=0.001 0.001 0.001; visual mesh filename=ABSOLUTE_PATH_TO_MESHES/sim_sea_2-5_l_upper_thigh_prt-binar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 scale=0.001 0.001 0.001
- link l_leg_jet_turbine: geometry collision mesh filename=ABSOLUTE_PATH_TO_TURBINES_MESHES/l_leg_jet_turbine.dae scale=0.001 0.001 0.001; visual mesh filename=ABSOLUTE_PATH_TO_TURBINES_MESHES/l_leg_jet_turbine.dae scale=0.001 0.001 0.001
- link l_leg_jet_turbine_prime: geometry collision mesh filename=ABSOLUTE_PATH_TO_TURBINES_MESHES/l_leg_jet_turbine.dae scale=0.001 0.001 0.001; visual mesh filename=ABSOLUTE_PATH_TO_TURBINES_MESHES/l_leg_jet_turbine.dae scale=0.001 0.001 0.001
- link l_lower_leg: geometry collision mesh filename=ABSOLUTE_PATH_TO_MESHES/sim_sea_2-5_l_shank_prt-binary.dae scale=0.001 0.001 0.001; visual mesh filename=ABSOLUTE_PATH_TO_MESHES/sim_sea_2-5_l_shank_prt-binary.dae scale=0.001 0.001 0.001
- link l_shoulder_1: geometry collision mesh filename=ABSOLUTE_PATH_TO_MESHES/sim_sea_2-5_l_shoulder_1_prt-binary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 scale=0.001 0.001 0.001; visual mesh filename=ABSOLUTE_PATH_TO_MESHES/sim_sea_2-5_l_shoulder_1_prt-binary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 scale=0.001 0.001 0.001
- link l_shoulder_2: geometry collision mesh filename=ABSOLUTE_PATH_TO_MESHES/sim_sea_2-5_l_shoulder_2_prt-binary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 scale=0.001 0.001 0.001; visual mesh filename=ABSOLUTE_PATH_TO_MESHES/sim_sea_2-5_l_shoulder_2_prt-binary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 scale=0.001 0.001 0.001
- link l_shoulder_3: geometry collision mesh filename=ABSOLUTE_PATH_TO_MESHES/sim_sea_2-5_l_upper_arm_prt-binary.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 scale=0.001 0.001 0.001; visual mesh filename=ABSOLUTE_PATH_TO_MESHES/sim_sea_2-5_l_upper_arm_prt-binary.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 scale=0.001 0.001 0.001
- link l_upper_arm: geometry collision mesh filename=ABSOLUTE_PATH_TO_MESHES/sim_sea_2-5_l_elbow_prt-binary.dae scale=0.001 0.001 0.001; visual mesh filename=ABSOLUTE_PATH_TO_MESHES/sim_sea_2-5_l_elbow_prt-binary.dae scale=0.001 0.001 0.001
- link l_upper_leg: geometry collision mesh filename=ABSOLUTE_PATH_TO_MESHES/sim_sea_2-5_l_thigh_prt-binary.dae scale=0.001 0.001 0.001; visual mesh filename=ABSOLUTE_PATH_TO_MESHES/sim_sea_2-5_l_thigh_prt-binary.dae scale=0.001 0.001 0.001
- link l_wrist_1: geometry collision mesh filename=ABSOLUTE_PATH_TO_MESHES/sim_sea_2-5_l_wrist_pitch_prt-binar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 scale=0.001 0.001 0.001; visual mesh filename=ABSOLUTE_PATH_TO_MESHES/sim_sea_2-5_l_wrist_pitch_prt-binar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 scale=0.001 0.001 0.001
- link neck_1: geometry collision mesh filename=ABSOLUTE_PATH_TO_MESHES/sim_sea_2-5_neck_1_prt-binary.dae scale=0.001 0.001 0.001; visual mesh filename=ABSOLUTE_PATH_TO_MESHES/sim_sea_2-5_neck_1_prt-binary.dae scale=0.001 0.001 0.001
- link neck_2: geometry collision mesh filename=ABSOLUTE_PATH_TO_MESHES/sim_sea_2-5_neck_2_prt-binary.dae scale=0.001 0.001 0.001; visual mesh filename=ABSOLUTE_PATH_TO_MESHES/sim_sea_2-5_neck_2_prt-binary.dae scale=0.001 0.001 0.001
- link r_ankle_1: geometry collision mesh filename=ABSOLUTE_PATH_TO_MESHES/sim_sea_2-5_r_ankle_prt-binary.dae scale=0.001 0.001 0.001; visual mesh filename=ABSOLUTE_PATH_TO_MESHES/sim_sea_2-5_r_ankle_prt-binary.dae scale=0.001 0.001 0.001
- link r_ankle_2: geometry collision mesh filename=ABSOLUTE_PATH_TO_MESHES/sim_sea_2-5_r_foot_prt-binary.dae scale=0.001 0.001 0.001; visual mesh filename=ABSOLUTE_PATH_TO_MESHES/sim_sea_2-5_r_foot_prt-binary.dae scale=0.001 0.001 0.001
- link r_arm_jet_turbine: geometry collision mesh filename=ABSOLUTE_PATH_TO_TURBINES_MESHES/r_arm_jet_turbine.dae scale=0.001 0.001 0.001; visual mesh filename=ABSOLUTE_PATH_TO_TURBINES_MESHES/r_arm_jet_turbine.dae scale=0.001 0.001 0.001
- link r_arm_jet_turbine_prime: geometry collision mesh filename=ABSOLUTE_PATH_TO_TURBINES_MESHES/r_arm_jet_turbine.dae scale=0.001 0.001 0.001; visual mesh filename=ABSOLUTE_PATH_TO_TURBINES_MESHES/r_arm_jet_turbine.dae scale=0.001 0.001 0.001
- link r_elbow_1: geometry collision mesh filename=ABSOLUTE_PATH_TO_MESHES/sim_sea_2-5_r_elbow_prosup_prt-bina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 scale=0.001 0.001 0.001; visual mesh filename=ABSOLUTE_PATH_TO_MESHES/sim_sea_2-5_r_elbow_prosup_prt-bina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 scale=0.001 0.001 0.001
- link r_foot: geometry collision box size=0.16 0.072 0.001; visual mesh filename=ABSOLUTE_PATH_TO_MESHES/sim_sea_2-5_r_sole_prt-binary.dae scale=0.001 0.001 0.001
- link r_forearm: geometry collision mesh filename=ABSOLUTE_PATH_TO_MESHES/sim_sea_2-5_r_forearm_prt-binary.dae scale=0.001 0.001 0.001; visual mesh filename=ABSOLUTE_PATH_TO_MESHES/sim_sea_2-5_r_forearm_prt-binary.dae scale=0.001 0.001 0.001
- link r_hand: geometry collision mesh filename=ABSOLUTE_PATH_TO_MESHES/sim_sea_2-5_r_hand_prt-binary.dae scale=0.001 0.001 0.001; visual mesh filename=ABSOLUTE_PATH_TO_MESHES/sim_sea_2-5_r_hand_prt-binary.dae scale=0.001 0.001 0.001
- link r_hip_1: geometry collision mesh filename=ABSOLUTE_PATH_TO_MESHES/sim_sea_2-5_r_hip_1_prt-binary.dae scale=0.001 0.001 0.001; visual mesh filename=ABSOLUTE_PATH_TO_MESHES/sim_sea_2-5_r_hip_1_prt-binary.dae scale=0.001 0.001 0.001
- link r_hip_2: geometry collision mesh filename=ABSOLUTE_PATH_TO_MESHES/sim_sea_2-5_r_hip_2_prt-binary.dae scale=0.001 0.001 0.001; visual mesh filename=ABSOLUTE_PATH_TO_MESHES/sim_sea_2-5_r_hip_2_prt-binary.dae scale=0.001 0.001 0.001
- link r_hip_3: geometry collision mesh filename=ABSOLUTE_PATH_TO_MESHES/sim_sea_2-5_r_upper_thigh_prt-binar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 scale=0.001 0.001 0.001; visual mesh filename=ABSOLUTE_PATH_TO_MESHES/sim_sea_2-5_r_upper_thigh_prt-binar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 scale=0.001 0.001 0.001
- link r_leg_jet_turbine: geometry collision mesh filename=ABSOLUTE_PATH_TO_TURBINES_MESHES/r_leg_jet_turbine.dae scale=0.001 0.001 0.001; visual mesh filename=ABSOLUTE_PATH_TO_TURBINES_MESHES/r_leg_jet_turbine.dae scale=0.001 0.001 0.001
- link r_leg_jet_turbine_prime: geometry collision mesh filename=ABSOLUTE_PATH_TO_TURBINES_MESHES/r_leg_jet_turbine.dae scale=0.001 0.001 0.001; visual mesh filename=ABSOLUTE_PATH_TO_TURBINES_MESHES/r_leg_jet_turbine.dae scale=0.001 0.001 0.001
- link r_lower_leg: geometry collision mesh filename=ABSOLUTE_PATH_TO_MESHES/sim_sea_2-5_r_shank_prt-binary.dae scale=0.001 0.001 0.001; visual mesh filename=ABSOLUTE_PATH_TO_MESHES/sim_sea_2-5_r_shank_prt-binary.dae scale=0.001 0.001 0.001
- link r_shoulder_1: geometry collision mesh filename=ABSOLUTE_PATH_TO_MESHES/sim_sea_2-5_r_shoulder_1_prt-binary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 scale=0.001 0.001 0.001; visual mesh filename=ABSOLUTE_PATH_TO_MESHES/sim_sea_2-5_r_shoulder_1_prt-binary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 scale=0.001 0.001 0.001
- link r_shoulder_2: geometry collision mesh filename=ABSOLUTE_PATH_TO_MESHES/sim_sea_2-5_r_shoulder_2_prt-binary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 scale=0.001 0.001 0.001; visual mesh filename=ABSOLUTE_PATH_TO_MESHES/sim_sea_2-5_r_shoulder_2_prt-binary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 scale=0.001 0.001 0.001
- link r_shoulder_3: geometry collision mesh filename=ABSOLUTE_PATH_TO_MESHES/sim_sea_2-5_r_upper_arm_prt-binary.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 scale=0.001 0.001 0.001; visual mesh filename=ABSOLUTE_PATH_TO_MESHES/sim_sea_2-5_r_upper_arm_prt-binary.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 scale=0.001 0.001 0.001
- link r_upper_arm: geometry collision mesh filename=ABSOLUTE_PATH_TO_MESHES/sim_sea_2-5_r_elbow_prt-binary.dae scale=0.001 0.001 0.001; visual mesh filename=ABSOLUTE_PATH_TO_MESHES/sim_sea_2-5_r_elbow_prt-binary.dae scale=0.001 0.001 0.001
- link r_upper_leg: geometry collision mesh filename=ABSOLUTE_PATH_TO_MESHES/sim_sea_2-5_r_thigh_prt-binary.dae scale=0.001 0.001 0.001; visual mesh filename=ABSOLUTE_PATH_TO_MESHES/sim_sea_2-5_r_thigh_prt-binary.dae scale=0.001 0.001 0.001
- link r_wrist_1: geometry collision mesh filename=ABSOLUTE_PATH_TO_MESHES/sim_sea_2-5_r_wrist_pitch_prt-binar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 scale=0.001 0.001 0.001; visual mesh filename=ABSOLUTE_PATH_TO_MESHES/sim_sea_2-5_r_wrist_pitch_prt-binar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 scale=0.001 0.001 0.001
- link root_link: geometry collision mesh filename=ABSOLUTE_PATH_TO_MESHES/sim_sea_2-5_root_link_prt-binary.dae scale=0.001 0.001 0.001; visual mesh filename=ABSOLUTE_PATH_TO_MESHES/sim_sea_2-5_root_link_prt-binary.dae scale=0.001 0.001 0.001
- link torso_1: geometry collision mesh filename=ABSOLUTE_PATH_TO_MESHES/sim_sea_2-5_lap_belt_1_prt-binary.d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 scale=0.001 0.001 0.001; visual mesh filename=ABSOLUTE_PATH_TO_MESHES/sim_sea_2-5_lap_belt_1_prt-binary.d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 scale=0.001 0.001 0.001
- link torso_2: geometry collision mesh filename=ABSOLUTE_PATH_TO_MESHES/sim_sea_2-5_lap_belt_2_prt-binary.d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 scale=0.001 0.001 0.001; visual mesh filename=ABSOLUTE_PATH_TO_MESHES/sim_sea_2-5_lap_belt_2_prt-binary.d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 scale=0.001 0.001 0.001

Commit message: fixed path to meshes

File: models/iCubGazeboV2_5/model.urdf (robot description, URDF)
Before this commit: robot iCub, 189 links, 188 joints
Links:
- link chest: geometry collision mesh filename=ABSOLUTE_PATH_TO_MESHES/sim_sea_2-5_chest_bb_prt-binary.dae scale=0.001 0.001 0.001; visual mesh filename=ABSOLUTE_PATH_TO_MESHES/sim_sea_2-5_chest_bb_prt-binary.dae scale=0.001 0.001 0.001
- link head: geometry collision mesh filename=ABSOLUTE_PATH_TO_MESHES/sim_sea_2-5_head_prt-binary.dae scale=0.001 0.001 0.001; visual mesh filename=ABSOLUTE_PATH_TO_MESHES/sim_sea_2-5_head_prt-binary.dae scale=0.001 0.001 0.001
- link l_ankle_1: geometry collision mesh filename=ABSOLUTE_PATH_TO_MESHES/sim_sea_2-5_l_ankle_prt-binary.dae scale=0.001 0.001 0.001; visual mesh filename=ABSOLUTE_PATH_TO_MESHES/sim_sea_2-5_l_ankle_prt-binary.dae scale=0.001 0.001 0.001
- link l_ankle_2: geometry collision mesh filename=ABSOLUTE_PATH_TO_MESHES/sim_sea_2-5_l_foot_prt-binary.dae scale=0.001 0.001 0.001; visual mesh filename=ABSOLUTE_PATH_TO_MESHES/sim_sea_2-5_l_foot_prt-binary.dae scale=0.001 0.001 0.001
- link l_elbow_1: geometry collision mesh filename=ABSOLUTE_PATH_TO_MESHES/sim_sea_2-5_l_elbow_prosup_prt-bina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 scale=0.001 0.001 0.001; visual mesh filename=ABSOLUTE_PATH_TO_MESHES/sim_sea_2-5_l_elbow_prosup_prt-bina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 scale=0.001 0.001 0.001
- link l_foot: geometry collision box size=0.16 0.072 0.001; visual mesh filename=ABSOLUTE_PATH_TO_MESHES/sim_sea_2-5_l_sole_prt-binary.dae scale=0.001 0.001 0.001
- link l_forearm: geometry collision mesh filename=ABSOLUTE_PATH_TO_MESHES/sim_sea_2-5_l_forearm_prt-binary.dae scale=0.001 0.001 0.001; visual mesh filename=ABSOLUTE_PATH_TO_MESHES/sim_sea_2-5_l_forearm_prt-binary.dae scale=0.001 0.001 0.001
- link l_hand: geometry collision mesh filename=ABSOLUTE_PATH_TO_MESHES/sim_sea_2-5_l_hand_prt-binary.dae scale=0.001 0.001 0.001; visual mesh filename=ABSOLUTE_PATH_TO_MESHES/sim_sea_2-5_l_hand_prt-binary.dae scale=0.001 0.001 0.001
- link l_hip_1: geometry collision mesh filename=ABSOLUTE_PATH_TO_MESHES/sim_sea_2-5_l_hip_1_prt-binary.dae scale=0.001 0.001 0.001; visual mesh filename=ABSOLUTE_PATH_TO_MESHES/sim_sea_2-5_l_hip_1_prt-binary.dae scale=0.001 0.001 0.001
- link l_hip_2: geometry collision mesh filename=ABSOLUTE_PATH_TO_MESHES/sim_sea_2-5_l_hip_2_prt-binary.dae scale=0.001 0.001 0.001; visual mesh filename=ABSOLUTE_PATH_TO_MESHES/sim_sea_2-5_l_hip_2_prt-binary.dae scale=0.001 0.001 0.001
- link l_hip_3: geometry collision mesh filename=ABSOLUTE_PATH_TO_MESHES/sim_sea_2-5_l_upper_thigh_prt-binar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 scale=0.001 0.001 0.001; visual mesh filename=ABSOLUTE_PATH_TO_MESHES/sim_sea_2-5_l_upper_thigh_prt-binar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 scale=0.001 0.001 0.001
- link l_lower_leg: geometry collision mesh filename=ABSOLUTE_PATH_TO_MESHES/sim_sea_2-5_l_shank_prt-binary.dae scale=0.001 0.001 0.001; visual mesh filename=ABSOLUTE_PATH_TO_MESHES/sim_sea_2-5_l_shank_prt-binary.dae scale=0.001 0.001 0.001
- link l_shoulder_1: geometry collision mesh filename=ABSOLUTE_PATH_TO_MESHES/sim_sea_2-5_l_shoulder_1_prt-binary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 scale=0.001 0.001 0.001; visual mesh filename=ABSOLUTE_PATH_TO_MESHES/sim_sea_2-5_l_shoulder_1_prt-binary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 scale=0.001 0.001 0.001
- link l_shoulder_2: geometry collision mesh filename=ABSOLUTE_PATH_TO_MESHES/sim_sea_2-5_l_shoulder_2_prt-binary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 scale=0.001 0.001 0.001; visual mesh filename=ABSOLUTE_PATH_TO_MESHES/sim_sea_2-5_l_shoulder_2_prt-binary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 scale=0.001 0.001 0.001
- link l_shoulder_3: geometry collision mesh filename=ABSOLUTE_PATH_TO_MESHES/sim_sea_2-5_l_upper_arm_prt-binary.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 scale=0.001 0.001 0.001; visual mesh filename=ABSOLUTE_PATH_TO_MESHES/sim_sea_2-5_l_upper_arm_prt-binary.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 scale=0.001 0.001 0.001
- link l_upper_arm: geometry collision mesh filename=ABSOLUTE_PATH_TO_MESHES/sim_sea_2-5_l_elbow_prt-binary.dae scale=0.001 0.001 0.001; visual mesh filename=ABSOLUTE_PATH_TO_MESHES/sim_sea_2-5_l_elbow_prt-binary.dae scale=0.001 0.001 0.001
- link l_upper_leg: geometry collision mesh filename=ABSOLUTE_PATH_TO_MESHES/sim_sea_2-5_l_thigh_prt-binary.dae scale=0.001 0.001 0.001; visual mesh filename=ABSOLUTE_PATH_TO_MESHES/sim_sea_2-5_l_thigh_prt-binary.dae scale=0.001 0.001 0.001
- link l_wrist_1: geometry collision mesh filename=ABSOLUTE_PATH_TO_MESHES/sim_sea_2-5_l_wrist_pitch_prt-binar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 scale=0.001 0.001 0.001; visual mesh filename=ABSOLUTE_PATH_TO_MESHES/sim_sea_2-5_l_wrist_pitch_prt-binar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 scale=0.001 0.001 0.001
- link neck_1: geometry collision mesh filename=ABSOLUTE_PATH_TO_MESHES/sim_sea_2-5_neck_1_prt-binary.dae scale=0.001 0.001 0.001; visual mesh filename=ABSOLUTE_PATH_TO_MESHES/sim_sea_2-5_neck_1_prt-binary.dae scale=0.001 0.001 0.001
- link neck_2: geometry collision mesh filename=ABSOLUTE_PATH_TO_MESHES/sim_sea_2-5_neck_2_prt-binary.dae scale=0.001 0.001 0.001; visual mesh filename=ABSOLUTE_PATH_TO_MESHES/sim_sea_2-5_neck_2_prt-binary.dae scale=0.001 0.001 0.001
- link r_ankle_1: geometry collision mesh filename=ABSOLUTE_PATH_TO_MESHES/sim_sea_2-5_r_ankle_prt-binary.dae scale=0.001 0.001 0.001; visual mesh filename=ABSOLUTE_PATH_TO_MESHES/sim_sea_2-5_r_ankle_prt-binary.dae scale=0.001 0.001 0.001
- link r_ankle_2: geometry collision mesh filename=ABSOLUTE_PATH_TO_MESHES/sim_sea_2-5_r_foot_prt-binary.dae scale=0.001 0.001 0.001; visual mesh filename=ABSOLUTE_PATH_TO_MESHES/sim_sea_2-5_r_foot_prt-binary.dae scale=0.001 0.001 0.001
- link r_elbow_1: geometry collision mesh filename=ABSOLUTE_PATH_TO_MESHES/sim_sea_2-5_r_elbow_prosup_prt-bina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 scale=0.001 0.001 0.001; visual mesh filename=ABSOLUTE_PATH_TO_MESHES/sim_sea_2-5_r_elbow_prosup_prt-bina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 scale=0.001 0.001 0.001
- link r_foot: geometry collision box size=0.16 0.072 0.001; visual mesh filename=ABSOLUTE_PATH_TO_MESHES/sim_sea_2-5_r_sole_prt-binary.dae scale=0.001 0.001 0.001
- link r_forearm: geometry collision mesh filename=ABSOLUTE_PATH_TO_MESHES/sim_sea_2-5_r_forearm_prt-binary.dae scale=0.001 0.001 0.001; visual mesh filename=ABSOLUTE_PATH_TO_MESHES/sim_sea_2-5_r_forearm_prt-binary.dae scale=0.001 0.001 0.001
- link r_hand: geometry collision mesh filename=ABSOLUTE_PATH_TO_MESHES/sim_sea_2-5_r_hand_prt-binary.dae scale=0.001 0.001 0.001; visual mesh filename=ABSOLUTE_PATH_TO_MESHES/sim_sea_2-5_r_hand_prt-binary.dae scale=0.001 0.001 0.001
- link r_hip_1: geometry collision mesh filename=ABSOLUTE_PATH_TO_MESHES/sim_sea_2-5_r_hip_1_prt-binary.dae scale=0.001 0.001 0.001; visual mesh filename=ABSOLUTE_PATH_TO_MESHES/sim_sea_2-5_r_hip_1_prt-binary.dae scale=0.001 0.001 0.001
- link r_hip_2: geometry collision mesh filename=ABSOLUTE_PATH_TO_MESHES/sim_sea_2-5_r_hip_2_prt-binary.dae scale=0.001 0.001 0.001; visual mesh filename=ABSOLUTE_PATH_TO_MESHES/sim_sea_2-5_r_hip_2_prt-binary.dae scale=0.001 0.001 0.001
- link r_hip_3: geometry collision mesh filename=ABSOLUTE_PATH_TO_MESHES/sim_sea_2-5_r_upper_thigh_prt-binar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 scale=0.001 0.001 0.001; visual mesh filename=ABSOLUTE_PATH_TO_MESHES/sim_sea_2-5_r_upper_thigh_prt-binar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 scale=0.001 0.001 0.001
- link r_lower_leg: geometry collision mesh filename=ABSOLUTE_PATH_TO_MESHES/sim_sea_2-5_r_shank_prt-binary.dae scale=0.001 0.001 0.001; visual mesh filename=ABSOLUTE_PATH_TO_MESHES/sim_sea_2-5_r_shank_prt-binary.dae scale=0.001 0.001 0.001
- link r_shoulder_1: geometry collision mesh filename=ABSOLUTE_PATH_TO_MESHES/sim_sea_2-5_r_shoulder_1_prt-binary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 scale=0.001 0.001 0.001; visual mesh filename=ABSOLUTE_PATH_TO_MESHES/sim_sea_2-5_r_shoulder_1_prt-binary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 scale=0.001 0.001 0.001
- link r_shoulder_2: geometry collision mesh filename=ABSOLUTE_PATH_TO_MESHES/sim_sea_2-5_r_shoulder_2_prt-binary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 scale=0.001 0.001 0.001; visual mesh filename=ABSOLUTE_PATH_TO_MESHES/sim_sea_2-5_r_shoulder_2_prt-binary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 scale=0.001 0.001 0.001
- link r_shoulder_3: geometry collision mesh filename=ABSOLUTE_PATH_TO_MESHES/sim_sea_2-5_r_upper_arm_prt-binary.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 scale=0.001 0.001 0.001; visual mesh filename=ABSOLUTE_PATH_TO_MESHES/sim_sea_2-5_r_upper_arm_prt-binary.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 scale=0.001 0.001 0.001
- link r_upper_arm: geometry collision mesh filename=ABSOLUTE_PATH_TO_MESHES/sim_sea_2-5_r_elbow_prt-binary.dae scale=0.001 0.001 0.001; visual mesh filename=ABSOLUTE_PATH_TO_MESHES/sim_sea_2-5_r_elbow_prt-binary.dae scale=0.001 0.001 0.001
- link r_upper_leg: geometry collision mesh filename=ABSOLUTE_PATH_TO_MESHES/sim_sea_2-5_r_thigh_prt-binary.dae scale=0.001 0.001 0.001; visual mesh filename=ABSOLUTE_PATH_TO_MESHES/sim_sea_2-5_r_thigh_prt-binary.dae scale=0.001 0.001 0.001
- link r_wrist_1: geometry collision mesh filename=ABSOLUTE_PATH_TO_MESHES/sim_sea_2-5_r_wrist_pitch_prt-binar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 scale=0.001 0.001 0.001; visual mesh filename=ABSOLUTE_PATH_TO_MESHES/sim_sea_2-5_r_wrist_pitch_prt-binar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 scale=0.001 0.001 0.001
- link root_link: geometry collision mesh filename=ABSOLUTE_PATH_TO_MESHES/sim_sea_2-5_root_link_prt-binary.dae scale=0.001 0.001 0.001; visual mesh filename=ABSOLUTE_PATH_TO_MESHES/sim_sea_2-5_root_link_prt-binary.dae scale=0.001 0.001 0.001
- link torso_1: geometry collision mesh filename=ABSOLUTE_PATH_TO_MESHES/sim_sea_2-5_lap_belt_1_prt-binary.d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 scale=0.001 0.001 0.001; visual mesh filename=ABSOLUTE_PATH_TO_MESHES/sim_sea_2-5_lap_belt_1_prt-binary.d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 scale=0.001 0.001 0.001
- link torso_2: geometry collision mesh filename=ABSOLUTE_PATH_TO_MESHES/sim_sea_2-5_lap_belt_2_prt-binary.d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 scale=0.001 0.001 0.001; visual mesh filename=ABSOLUTE_PATH_TO_MESHES/sim_sea_2-5_lap_belt_2_prt-binary.d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 scale=0.001 0.001 0.001
