Commit message: models updated for the new iDynTree visualizer

File: models/iCubGazeboV2_5/model.urdf (robot description, URDF)
Before this commit: robot iCub, 189 links, 188 joints
Links:
- link chest: geometry collision mesh filename=package://meshes/sim_sea_2-5_chest_bb_prt-binary.stl scale=0.001 0.001 0.001; visual mesh filename=package://meshes/sim_sea_2-5_chest_bb_prt-binary.stl scale=0.001 0.001 0.001
- link head: geometry collision mesh filename=package://meshes/sim_sea_2-5_head_prt-binary.stl scale=0.001 0.001 0.001; visual mesh filename=package://meshes/sim_sea_2-5_head_prt-binary.stl scale=0.001 0.001 0.001
- link l_ankle_1: geometry collision mesh filename=package://meshes/sim_sea_2-5_l_ankle_prt-binary.stl scale=0.001 0.001 0.001; visual mesh filename=package://meshes/sim_sea_2-5_l_ankle_prt-binary.stl scale=0.001 0.001 0.001
- link l_ankle_2: geometry collision mesh filename=package://meshes/sim_sea_2-5_l_foot_prt-binary.stl scale=0.001 0.001 0.001; visual mesh filename=package://meshes/sim_sea_2-5_l_foot_prt-binary.stl scale=0.001 0.001 0.001
- link l_elbow_1: geometry collision mesh filename=package://meshes/sim_sea_2-5_l_elbow_prosup_prt-binary.stl scale=0.001 0.001 0.001; visual mesh filename=package://meshes/sim_sea_2-5_l_elbow_prosup_prt-binary.stl scale=0.001 0.001 0.001
- link l_foot: geometry collision box size=0.16 0.072 0.001; visual mesh filename=package://meshes/sim_sea_2-5_l_sole_prt-binary.stl scale=0.001 0.001 0.001
- link l_forearm: geometry collision mesh filename=package://meshes/sim_sea_2-5_l_forearm_prt-binary.stl scale=0.001 0.001 0.001; visual mesh filename=package://meshes/sim_sea_2-5_l_forearm_prt-binary.stl scale=0.001 0.001 0.001
- link l_hand: geometry collision mesh filename=package://meshes/sim_sea_2-5_l_hand_prt-binary.stl scale=0.001 0.001 0.001; visual mesh filename=package://meshes/sim_sea_2-5_l_hand_prt-binary.stl scale=0.001 0.001 0.001
- link l_hip_1: geometry collision mesh filename=package://meshes/sim_sea_2-5_l_hip_1_prt-binary.stl scale=0.001 0.001 0.001; visual mesh filename=package://meshes/sim_sea_2-5_l_hip_1_prt-binary.stl scale=0.001 0.001 0.001
- link l_hip_2: geometry collision mesh filename=package://meshes/sim_sea_2-5_l_hip_2_prt-binary.stl scale=0.001 0.001 0.001; visual mesh filename=package://meshes/sim_sea_2-5_l_hip_2_prt-binary.stl scale=0.001 0.001 0.001
- link l_hip_3: geometry collision mesh filename=package://meshes/sim_sea_2-5_l_upper_thigh_prt-binary.stl scale=0.001 0.001 0.001; visual mesh filename=package://meshes/sim_sea_2-5_l_upper_thigh_prt-binary.stl scale=0.001 0.001 0.001
- link l_lower_leg: geometry collision mesh filename=package://meshes/sim_sea_2-5_l_shank_prt-binary.stl scale=0.001 0.001 0.001; visual mesh filename=package://meshes/sim_sea_2-5_l_shank_prt-binary.stl scale=0.001 0.001 0.001
- link l_shoulder_1: geometry collision mesh filename=package://meshes/sim_sea_2-5_l_shoulder_1_prt-binary.stl scale=0.001 0.001 0.001; visual mesh filename=package://meshes/sim_sea_2-5_l_shoulder_1_prt-binary.stl scale=0.001 0.001 0.001
- link l_shoulder_2: geometry collision mesh filename=package://meshes/sim_sea_2-5_l_shoulder_2_prt-binary.stl scale=0.001 0.001 0.001; visual mesh filename=package://meshes/sim_sea_2-5_l_shoulder_2_prt-binary.stl scale=0.001 0.001 0.001
- link l_shoulder_3: geometry collision mesh filename=package://meshes/sim_sea_2-5_l_upper_arm_prt-binary.stl scale=0.001 0.001 0.001; visual mesh filename=package://meshes/sim_sea_2-5_l_upper_arm_prt-binary.stl scale=0.001 0.001 0.001
- link l_upper_arm: geometry collision mesh filename=package://meshes/sim_sea_2-5_l_elbow_prt-binary.stl scale=0.001 0.001 0.001; visual mesh filename=package://meshes/sim_sea_2-5_l_elbow_prt-binary.stl scale=0.001 0.001 0.001
- link l_upper_leg: geometry collision mesh filename=package://meshes/sim_sea_2-5_l_thigh_prt-binary.stl scale=0.001 0.001 0.001; visual mesh filename=package://meshes/sim_sea_2-5_l_thigh_prt-binary.stl scale=0.001 0.001 0.001
- link l_wrist_1: geometry collision mesh filename=package://meshes/sim_sea_2-5_l_wrist_pitch_prt-binary.stl scale=0.001 0.001 0.001; visual mesh filename=package://meshes/sim_sea_2-5_l_wrist_pitch_prt-binary.stl scale=0.001 0.001 0.001
- link neck_1: geometry collision mesh filename=package://meshes/sim_sea_2-5_neck_1_prt-binary.stl scale=0.001 0.001 0.001; visual mesh filename=package://meshes/sim_sea_2-5_neck_1_prt-binary.stl scale=0.001 0.001 0.001
- link neck_2: geometry collision mesh filename=package://meshes/sim_sea_2-5_neck_2_prt-binary.stl scale=0.001 0.001 0.001; visual mesh filename=package://meshes/sim_sea_2-5_neck_2_prt-binary.stl scale=0.001 0.001 0.001
- link r_ankle_1: geometry collision mesh filename=package://meshes/sim_sea_2-5_r_ankle_prt-binary.stl scale=0.001 0.001 0.001; visual mesh filename=package://meshes/sim_sea_2-5_r_ankle_prt-binary.stl scale=0.001 0.001 0.001
- link r_ankle_2: geometry collision mesh filename=package://meshes/sim_sea_2-5_r_foot_prt-binary.stl scale=0.001 0.001 0.001; visual mesh filename=package://meshes/sim_sea_2-5_r_foot_prt-binary.stl scale=0.001 0.001 0.001
- link r_elbow_1: geometry collision mesh filename=package://meshes/sim_sea_2-5_r_elbow_prosup_prt-binary.stl scale=0.001 0.001 0.001; visual mesh filename=package://meshes/sim_sea_2-5_r_elbow_prosup_prt-binary.stl scale=0.001 0.001 0.001
- link r_foot: geometry collision box size=0.16 0.072 0.001; visual mesh filename=package://meshes/sim_sea_2-5_r_sole_prt-binary.stl scale=0.001 0.001 0.001
- link r_forearm: geometry collision mesh filename=package://meshes/sim_sea_2-5_r_forearm_prt-binary.stl scale=0.001 0.001 0.001; visual mesh filename=package://meshes/sim_sea_2-5_r_forearm_prt-binary.stl scale=0.001 0.001 0.001
- link r_hand: geometry collision mesh filename=package://meshes/sim_sea_2-5_r_hand_prt-binary.stl scale=0.001 0.001 0.001; visual mesh filename=package://meshes/sim_sea_2-5_r_hand_prt-binary.stl scale=0.001 0.001 0.001
- link r_hip_1: geometry collision mesh filename=package://meshes/sim_sea_2-5_r_hip_1_prt-binary.stl scale=0.001 0.001 0.001; visual mesh filename=package://meshes/sim_sea_2-5_r_hip_1_prt-binary.stl scale=0.001 0.001 0.001
- link r_hip_2: geometry collision mesh filename=package://meshes/sim_sea_2-5_r_hip_2_prt-binary.stl scale=0.001 0.001 0.001; visual mesh filename=package://meshes/sim_sea_2-5_r_hip_2_prt-binary.stl scale=0.001 0.001 0.001
- link r_hip_3: geometry collision mesh filename=package://meshes/sim_sea_2-5_r_upper_thigh_prt-binary.stl scale=0.001 0.001 0.001; visual mesh filename=package://meshes/sim_sea_2-5_r_upper_thigh_prt-binary.stl scale=0.001 0.001 0.001
- link r_lower_leg: geometry collision mesh filename=package://meshes/sim_sea_2-5_r_shank_prt-binary.stl scale=0.001 0.001 0.001; visual mesh filename=package://meshes/sim_sea_2-5_r_shank_prt-binary.stl scale=0.001 0.001 0.001
- link r_shoulder_1: geometry collision mesh filename=package://meshes/sim_sea_2-5_r_shoulder_1_prt-binary.stl scale=0.001 0.001 0.001; visual mesh filename=package://meshes/sim_sea_2-5_r_shoulder_1_prt-binary.stl scale=0.001 0.001 0.001
- link r_shoulder_2: geometry collision mesh filename=package://meshes/sim_sea_2-5_r_shoulder_2_prt-binary.stl scale=0.001 0.001 0.001; visual mesh filename=package://meshes/sim_sea_2-5_r_shoulder_2_prt-binary.stl scale=0.001 0.001 0.001
- link r_shoulder_3: geometry collision mesh filename=package://meshes/sim_sea_2-5_r_upper_arm_prt-binary.stl scale=0.001 0.001 0.001; visual mesh filename=package://meshes/sim_sea_2-5_r_upper_arm_prt-binary.stl scale=0.001 0.001 0.001
- link r_upper_arm: geometry collision mesh filename=package://meshes/sim_sea_2-5_r_elbow_prt-binary.stl scale=0.001 0.001 0.001; visual mesh filename=package://meshes/sim_sea_2-5_r_elbow_prt-binary.stl scale=0.001 0.001 0.001
- link r_upper_leg: geometry collision mesh filename=package://meshes/sim_sea_2-5_r_thigh_prt-binary.stl scale=0.001 0.001 0.001; visual mesh filename=package://meshes/sim_sea_2-5_r_thigh_prt-binary.stl scale=0.001 0.001 0.001
- link r_wrist_1: geometry collision mesh filename=package://meshes/sim_sea_2-5_r_wrist_pitch_prt-binary.stl scale=0.001 0.001 0.001; visual mesh filename=package://meshes/sim_sea_2-5_r_wrist_pitch_prt-binary.stl scale=0.001 0.001 0.001
- link root_link: geometry collision mesh filename=package://meshes/sim_sea_2-5_root_link_prt-binary.stl scale=0.001 0.001 0.001; visual mesh filename=package://meshes/sim_sea_2-5_root_link_prt-binary.stl scale=0.001 0.001 0.001
- link torso_1: geometry collision mesh filename=package://meshes/sim_sea_2-5_lap_belt_1_prt-binary.stl scale=0.001 0.001 0.001; visual mesh filename=package://meshes/sim_sea_2-5_lap_belt_1_prt-binary.stl scale=0.001 0.001 0.001
- link torso_2: geometry collision mesh filename=package://meshes/sim_sea_2-5_lap_belt_2_prt-binary.stl scale=0.001 0.001 0.001; visual mesh filename=package://meshes/sim_sea_2-5_lap_belt_2_prt-binary.stl scale=0.001 0.001 0.001

File: models/icubGazeboSim/model.urdf (robot description, URDF)
Before this commit: robot iCub, 56 links, 55 joints
Links:
- link chest: geometry collision mesh filename=package://meshes/icub_simple_collision_chest.stl scale=1 1 1; visual mesh filename=package://meshes/icub_simple_collision_chest.stl scale=1 1 1
- link head: geometry collision mesh filename=package://meshes/icub_simple_collision_head.stl scale=1 1 1; visual mesh filename=package://meshes/icub_simple_collision_head.stl scale=1 1 1
- link l_ankle_1: geometry collision mesh filename=package://meshes/icub_simple_collision_l_ankle_1.stl scale=1 1 1; visual mesh filename=package://meshes/icub_simple_collision_l_ankle_1.stl scale=1 1 1
- link l_foot: geometry collision mesh filename=package://meshes/icub_simple_collision_l_foot.stl scale=1 1 1; visual mesh filename=package://meshes/icub_simple_collision_l_foot.stl scale=1 1 1
- link l_forearm: geometry collision mesh filename=package://meshes/icub_simple_collision_l_forearm.stl scale=1 1 1; visual mesh filename=package://meshes/icub_simple_collision_l_forearm.stl scale=1 1 1
- link l_hand: geometry collision mesh filename=package://meshes/icub_simple_collision_l_hand.stl scale=1 1 1; visual mesh filename=package://meshes/icub_simple_collision_l_hand.stl scale=1 1 1
- link l_hip_1: geometry collision mesh filename=package://meshes/icub_simple_collision_l_hip_1.stl scale=1 1 1; visual mesh filename=package://meshes/icub_simple_collision_l_hip_1.stl scale=1 1 1
- link l_hip_2: geometry collision mesh filename=package://meshes/icub_simple_collision_l_hip_2.stl scale=1 1 1; visual mesh filename=package://meshes/icub_simple_collision_l_hip_2.stl scale=1 1 1
- link l_lower_leg: geometry collision mesh filename=package://meshes/icub_simple_collision_l_shank.stl scale=1 1 1; visual mesh filename=package://meshes/icub_simple_collision_l_shank.stl scale=1 1 1
- link l_shoulder_1: geometry collision mesh filename=package://meshes/icub_simple_collision_l_shoulder_1.stl scale=1 1 1; visual mesh filename=package://meshes/icub_simple_collision_l_shoulder_1.stl scale=1 1 1
- link l_shoulder_2: geometry collision mesh filename=package://meshes/icub_simple_collision_l_shoulder_2.stl scale=1 1 1; visual mesh filename=package://meshes/icub_simple_collision_l_shoulder_2.stl scale=1 1 1
- link l_upper_arm: geometry collision mesh filename=package://meshes/icub_simple_collision_l_arm.stl scale=1 1 1; visual mesh filename=package://meshes/icub_simple_collision_l_arm.stl scale=1 1 1
- link l_upper_leg: geometry collision mesh filename=package://meshes/icub_simple_collision_l_thigh.stl scale=1 1 1; visual mesh filename=package://meshes/icub_simple_collision_l_thigh.stl scale=1 1 1
- link neck_1: geometry collision mesh filename=package://meshes/icub_simple_collision_neck_1.stl scale=1 1 1; visual mesh filename=package://meshes/icub_simple_collision_neck_1.stl scale=1 1 1
- link neck_2: geometry collision mesh filename=package://meshes/icub_simple_collision_neck_2.stl scale=1 1 1; visual mesh filename=package://meshes/icub_simple_collision_neck_2.stl scale=1 1 1
- link r_ankle_1: geometry collision mesh filename=package://meshes/icub_simple_collision_r_ankle_1.stl scale=1 1 1; visual mesh filename=package://meshes/icub_simple_collision_r_ankle_1.stl scale=1 1 1
- link r_foot: geometry collision mesh filename=package://meshes/icub_simple_collision_r_foot.stl scale=1 1 1; visual mesh filename=package://meshes/icub_simple_collision_r_foot.stl scale=1 1 1
- link r_forearm: geometry collision mesh filename=package://meshes/icub_simple_collision_r_forearm.stl scale=1 1 1; visual mesh filename=package://meshes/icub_simple_collision_r_forearm.stl scale=1 1 1
- link r_hand: geometry collision mesh filename=package://meshes/icub_simple_collision_r_hand.stl scale=1 1 1; visual mesh filename=package://meshes/icub_simple_collision_r_hand.stl scale=1 1 1
- link r_hip_1: geometry collision mesh filename=package://meshes/icub_simple_collision_r_hip_1.stl scale=1 1 1; visual mesh filename=package://meshes/icub_simple_collision_r_hip_1.stl scale=1 1 1
- link r_hip_2: geometry collision mesh filename=package://meshes/icub_simple_collision_r_hip_2.stl scale=1 1 1; visual mesh filename=package://meshes/icub_simple_collision_r_hip_2.stl scale=1 1 1
- link r_lower_leg: geometry collision mesh filename=package://meshes/icub_simple_collision_r_shank.stl scale=1 1 1; visual mesh filename=package://meshes/icub_simple_collision_r_shank.stl scale=1 1 1
- link r_shoulder_1: geometry collision mesh filename=package://meshes/icub_simple_collision_r_shoulder_1.stl scale=1 1 1; visual mesh filename=package://meshes/icub_simple_collision_r_shoulder_1.stl scale=1 1 1
- link r_shoulder_2: geometry collision mesh filename=package://meshes/icub_simple_collision_r_shoulder_2.stl scale=1 1 1; visual mesh filename=package://meshes/icub_simple_collision_r_shoulder_2.stl scale=1 1 1
- link r_upper_arm: geometry collision mesh filename=package://meshes/icub_simple_collision_r_arm.stl scale=1 1 1; visual mesh filename=package://meshes/icub_simple_collision_r_arm.stl scale=1 1 1
- link r_upper_leg: geometry collision mesh filename=package://meshes/icub_simple_collision_r_thigh.stl scale=1 1 1; visual mesh filename=package://meshes/icub_simple_collision_r_thigh.stl scale=1 1 1
- link root_link: geometry collision mesh filename=package://meshes/icub_simple_collision_root_link.stl scale=1 1 1; visual mesh filename=package://meshes/icub_simple_collision_root_link.stl scale=1 1 1
- link torso_1: geometry collision mesh filename=package://meshes/icub_simple_collision_lap_belt_1.stl scale=1 1 1; visual mesh filename=package://meshes/icub_simple_collision_lap_belt_1.stl scale=1 1 1
